Commit message: 24-04

File: urdf/robot_rrr_mod.urdf (robot description, URDF)
Before this commit: robot robot, 4 links, 3 joints
Links:
- link shoulder_link: geometry visual mesh filename=cubo.stl scale=0.010 0.010 0.010
Joints:
- joint arm_joint: origin xyz=0.3 0 0 rpy=0 0 0 -> xyz=0 0 0 rpy=1.57 0 0
- joint shoulder_joint: origin xyz=0 0 0 rpy=1.57 0 0 -> xyz=0 0 0.3 rpy=0 0 0
