Commit message: 27-04

File: urdf/robot_rrr.urdf (robot description, URDF)
Before this commit: robot robot, 4 links, 3 joints
Joints:
- joint arm_joint: limit lower=-3.14 upper=3.14 -> lower=-3.14 upper=3.14 effort=10.0 velocity=10.0
- joint forearm_joint: limit lower=-3.14 upper=3.14 -> lower=-3.14 upper=3.14 effort=10.0 velocity=10.0
- joint shoulder_joint: limit lower=-3.14 upper=3.14 -> lower=-3.14 upper=3.14 effort=10.0 velocity=10.0
